Commit message: urdf del rover

File: src/osr-rover-code/ROS/osr_gazebo/urdf/gazebo.urdf.xacro (robot description, xacro)
@@ -3,5 +3,5 @@
   <ros2_control name="GazeboSystem" type="system">
     <hardware>
-      <plugin>gazebo_ros2_control/GazeboSystem</plugin>
+      <plugin>gz_ros2_control/GazeboSimSystem</plugin>
     </hardware>
     <joint name="middle_wheel_joint_left">
@@ -112,27 +112,44 @@
   </ros2_control>
   <gazebo>
-    <plugin filename="libgazebo_ros2_control.so" name="gazebo_ros2_control">
+    <plugin filename="gz_ros2_control-system" name="gz_ros2_control::GazeboSimROS2ControlPlugin">
       <parameters>$(find osr_gazebo)/config/controller_velocity.yaml</parameters>
     </plugin>
   </gazebo>
-    <gazebo reference="imu_link">
-        <gravity>true</gravity>
-        <sensor name="imu_sensor" type="imu">
-        <always_on>true</always_on>
-        <update_rate>100</update_rate>
-        <visualize>true</visualize>
-        <topic>"imu"</topic>
-        <plugin filename="libgazebo_ros_imu_sensor.so" name="imu_plugin">
-            <topicName>imu</topicName>
-            <bodyName>imu_link</bodyName>
-            <updateRateHZ>100.0</updateRateHZ>
-            <gaussianNoise>0.0</gaussianNoise>
-            <xyzOffset>0 0 0</xyzOffset>
-            <rpyOffset>0 0 0</rpyOffset>
-            <frameName>imu_link</frameName>
-            <initialOrientationAsReference>false</initialOrientationAsReference>
-        </plugin>
-        <pose>0 0 0 0 0 0</pose>
-        </sensor>
-    </gazebo>
+  <gazebo reference="imu_link">
+      <sensor name="imu_sensor" type="imu">
+          <always_on>true</always_on>
+          <update_rate>100</update_rate>
+          <visualize>true</visualize>
+          <topic>imu</topic>
+          <gz_frame_id>imu_link</gz_frame_id>
+      </sensor>
+  </gazebo>
+  <gazebo reference="laser_frame">
+      <sensor name="laser" type="gpu_lidar">
+          <pose>0 0 0 0 0 0</pose>
+          <visualize>false</visualize> <update_rate>10</update_rate>
+          <topic>scan</topic>
+          <gz_frame_id>laser_frame</gz_frame_id>
+          <ray>
+              <scan>
+                  <horizontal>
+                      <samples>400</samples>
+                      <resolution>1</resolution>
+                      <min_angle>-3.14159</min_angle>
+                      <max_angle>3.14159</max_angle>
+                  </horizontal>
+              </scan>
+              <range>
+                  <min>0.15</min>
+                  <max>12.0</max>
+                  <resolution>0.01</resolution>
+              </range>
+              <noise>
+                  <type>gaussian</type>
+                  <mean>0.0</mean>
+                  <stddev>0.01</stddev>
+              </noise>
+          </ray>
+      </sensor>
+  </gazebo>
 </robot>

File: src/osr-rover-code/ROS/osr_gazebo/urdf/insert_transmission.urdf.xacro (robot description, xacro)
@@ -3,39 +3,27 @@
     <xacro:macro name="insert_effort_transmission" params="name">
         <transmission name="${name}_tran">
-            <type>transmission_interface/SimpleTransmission</type>
-            <joint name="${name}">
-                <hardwareInterface>EffortJointInterface</hardwareInterface>  <!-- Updated for ROS2 -->
-                <mechanicalReduction>1</mechanicalReduction>
+            <plugin>transmission_interface/SimpleTransmission</plugin>
+            <actuator name="${name}_motor" role="actuator1"/>
+            <joint name="${name}" role="joint1">
+                <mechanical_reduction>1.0</mechanical_reduction>
             </joint>
-            <actuator name="${name}_motor">
-                <hardwareInterface>EffortJointInterface</hardwareInterface>  <!-- Updated for ROS2 -->
-                <mechanicalReduction>1</mechanicalReduction>
-            </actuator>
         </transmission>
     </xacro:macro>
     <xacro:macro name="insert_position_transmission" params="name">
         <transmission name="${name}_tran">
-            <type>transmission_interface/SimpleTransmission</type>
-            <joint name="${name}">
-                <hardwareInterface>PositionJointInterface</hardwareInterface>  <!-- Updated for ROS2 -->
-                <mechanicalReduction>1</mechanicalReduction>
+            <plugin>transmission_interface/SimpleTransmission</plugin>
+            <actuator name="${name}_motor" role="actuator1"/>
+            <joint name="${name}" role="joint1">
+                <mechanical_reduction>1.0</mechanical_reduction>
             </joint>
-            <actuator name="${name}_motor">
-                <hardwareInterface>PositionJointInterface</hardwareInterface>  <!-- Updated for ROS2 -->
-                <mechanicalReduction>1</mechanicalReduction>
-            </actuator>
         </transmission>
     </xacro:macro>
     <xacro:macro name="insert_velocity_transmission" params="name">
         <transmission name="${name}_tran">
-            <type>transmission_interface/SimpleTransmission</type>
-            <joint name="${name}">
-                <hardwareInterface>VelocityJointInterface</hardwareInterface>  <!-- Updated for ROS2 -->
-                <mechanicalReduction>1</mechanicalReduction>
+            <plugin>transmission_interface/SimpleTransmission</plugin>
+            <actuator name="${name}_motor" role="actuator1"/>
+            <joint name="${name}" role="joint1">
+                <mechanical_reduction>1.0</mechanical_reduction>
             </joint>
-            <actuator name="${name}_motor">
-                <hardwareInterface>VelocityJointInterface</hardwareInterface>  <!-- Updated for ROS2 -->
-                <mechanicalReduction>1</mechanicalReduction>
-            </actuator>
         </transmission>
     </xacro:macro>

File: src/osr-rover-code/ROS/osr_gazebo/urdf/osr.urdf.xacro (robot description, xacro)
@@ -33,8 +33,8 @@
             <material name="brown"/>
         </visual>
-	    <inertial>
+        <inertial>
             <origin rpy="0 0 0" xyz="0 0 0"/>
             <mass value="10"/>
-            <inertia  ixx="0.28541666666666665" ixy="0" ixz="0" iyy="0.8666666666666666" 	iyz="0" izz="1.0854166666666665" />
+            <inertia  ixx="0.28541666666666665" ixy="0" ixz="0" iyy="0.8666666666666666"    iyz="0" izz="1.0854166666666665" />
         </inertial>
     </link>
@@ -241,5 +241,4 @@
         </link>
         <joint name="front_wheel_joint_${prefix}" type="revolute">
-        <!-- revolute continuous -->
             <parent link="rocker_bogie_link_${prefix}_2"/>
             <origin rpy="0 0 0" xyz="0.170113 -0.000335 0.076721"/>
@@ -295,5 +294,4 @@
         </link>
         <joint name="rear_wheel_joint_${prefix}" type="revolute">
-        <!-- revolute continuous -->
             <parent link="rocker_bogie_link_${prefix}_1"/>
             <origin rpy="0 0 0" xyz="-0.311763 0 -0.030379"/>
@@ -312,12 +310,4 @@
                     <mesh filename="file://$(find osr_gazebo)/meshes/wheel.stl"/>
                 </geometry>
-                <surface>
-                    <friction>
-                        <ode>
-                            <mu>0.7</mu>
-                            <mu2>0.3</mu2>
-                        </ode>
-                    </friction>
-                </surface>
             </collision>
             <visual>
@@ -334,4 +324,8 @@
             </inertial>
         </link>
+        <gazebo reference="front_wheel_link_${prefix}">
+            <mu1>0.7</mu1>
+            <mu2>0.3</mu2>
+        </gazebo>
         <joint name="front_wheel_joint_${prefix}" type="continuous">
             <parent link="front_wheel_link_${prefix_1}"/>
@@ -347,12 +341,4 @@
                     <mesh filename="file://$(find osr_gazebo)/meshes/wheel.stl"/>
                 </geometry>
-                <surface>
-                    <friction>
-                        <ode>
-                            <mu>0.7</mu>
-                            <mu2>0.3</mu2>
-                        </ode>
-                    </friction>
-                </surface>
             </collision>
             <visual>
@@ -369,4 +355,8 @@
             </inertial>
         </link>
+        <gazebo reference="middle_wheel_link_${prefix}">
+            <mu1>0.7</mu1>
+            <mu2>0.3</mu2>
+        </gazebo>
         <joint name="middle_wheel_joint_${prefix}" type="continuous">
             <parent link="middle_wheel_link_${prefix_1}"/>
@@ -382,12 +372,4 @@
                     <mesh filename="file://$(find osr_gazebo)/meshes/wheel.stl"/>
                 </geometry>
-                <surface>
-                    <friction>
-                        <ode>
-                            <mu>0.7</mu>
-                            <mu2>0.3</mu2>
-                        </ode>
-                    </friction>
-                </surface>
             </collision>
             <visual>
@@ -404,4 +386,8 @@
             </inertial>
         </link>
+        <gazebo reference="rear_wheel_link_${prefix}">
+            <mu1>0.7</mu1>
+            <mu2>0.3</mu2>
+        </gazebo>
         <joint name="rear_wheel_joint_${prefix}" type="continuous">
             <parent link="rear_wheel_link_${prefix_1}"/>
@@ -415,9 +401,28 @@
     <xacro:wheel prefix="right" dir="-1" origin="3.14" prefix_1="R"/>
     <joint name="imu_joint" type="fixed">
-            <parent link="base_link"/>
-            <child link="imu_link"/>
+        <parent link="base_link"/>
+        <child link="imu_link"/>
+        <origin xyz="0 0 0" rpy="0 0 0"/>
+    </joint>
+    <link name="imu_link"></link>
+    <link name="laser_frame">
+        <visual>
+            <geometry>
+                <cylinder radius="0.03" length="0.04"/>
+            </geometry>
             <origin xyz="0 0 0" rpy="0 0 0"/>
-        </joint>
-    <link name="imu_link"></link>
+        </visual>
+        <collision>
+            <geometry>
+                <cylinder radius="0.03" length="0.04"/>
+            </geometry>
+            <origin xyz="0 0 0" rpy="0 0 0"/>
+        </collision>
+    </link>
+    <joint name="laser_joint" type="fixed">
+        <parent link="base_link" />
+        <child link="laser_frame" />
+        <origin xyz="0.09 0 0.08" rpy="0 0 0" />
+    </joint>
     <xacro:insert_velocity_transmission name="rear_wheel_joint_right"/>
     <xacro:insert_velocity_transmission name="rear_wheel_joint_left"/>

Commit message: urdf rover añadido en rviz tmb

File: src/osr-rover-code/ROS/osr_gazebo/urdf/gazebo.urdf.xacro (robot description, xacro)
@@ -110,4 +110,14 @@
       <state_interface name="effort"/>
     </joint>
+    <joint name="rocker_bogie_joint_L_2">
+      <state_interface name="position"/>
+      <state_interface name="velocity"/>
+      <state_interface name="effort"/>
+    </joint>
+    <joint name="rocker_bogie_joint_R_2">
+      <state_interface name="position"/>
+      <state_interface name="velocity"/>
+      <state_interface name="effort"/>
+    </joint>
   </ros2_control>
   <gazebo>
