Commit message: ajuste mapa y goal, no va orientacion

File: src/osr-rover-code/ROS/osr_gazebo/urdf/osr.urdf.xacro (robot description, xacro)
@@ -423,5 +423,5 @@
         <parent link="base_link" />
         <child link="laser_frame" />
-        <origin xyz="0.09 0 0.08" rpy="0 0 0" />
+        <origin xyz="0.09 0 0.2" rpy="0 0 0" />
     </joint>
     <xacro:insert_velocity_transmission name="rear_wheel_joint_right"/>

Commit message: Prueba para osr completo

File: src/osr-rover-code/ROS/osr_gazebo/urdf/osr.urdf.xacro (robot description, xacro)
@@ -214,4 +214,5 @@
             <child link="rocker_bogie_link_${prefix}_2"/>
             <limit effort="10000.0" velocity="1.0" lower="-0.5" upper="0.5"/>
+            <dynamics damping="50.0" friction="20.0"/>
             <axis xyz="0 1 0"/>
         </joint>
@@ -244,5 +245,6 @@
             <origin rpy="0 0 0" xyz="0.170113 -0.000335 0.076721"/>
             <child link="front_wheel_link_${prefix}"/>
-            <limit effort="100000.0" velocity="10" lower="-0.523599" upper="0.523599"/>
+            <limit effort="100000.0" velocity="10.0" lower="-0.523599" upper="0.523599"/>
+            <dynamics damping="20.0" friction="10.0"/>
             <axis xyz="0 0 1"/>
         </joint>
@@ -297,5 +299,6 @@
             <origin rpy="0 0 0" xyz="-0.311763 0 -0.030379"/>
             <child link="rear_wheel_link_${prefix}"/>
-            <limit effort="100000.0" velocity="3" lower="-0.523599" upper="0.523599"/>
+            <limit effort="100000.0" velocity="3.0" lower="-0.523599" upper="0.523599"/>
+            <dynamics damping="20.0" friction="10.0"/>
             <axis xyz="0 0 1"/>
         </joint>
@@ -325,6 +328,6 @@
         </link>
         <gazebo reference="front_wheel_link_${prefix}">
-            <mu1>2.0</mu1>
-            <mu2>2.0</mu2>
+            <mu1>0.7</mu1>
+            <mu2>0.05</mu2>
         </gazebo>
         <joint name="front_wheel_joint_${prefix}" type="continuous">
@@ -333,5 +336,5 @@
             <child link="front_wheel_link_${prefix}"/>
             <axis xyz="0 1 0"/>
-            <velocity>5.0</velocity>
+            <limit effort="100.0" velocity="5.0"/>
         </joint>
         <link name="middle_wheel_link_${prefix}">
@@ -356,6 +359,6 @@
         </link>
         <gazebo reference="middle_wheel_link_${prefix}">
-            <mu1>2.0</mu1>
-            <mu2>2.0</mu2>
+            <mu1>0.7</mu1>
+            <mu2>0.05</mu2>
         </gazebo>
         <joint name="middle_wheel_joint_${prefix}" type="continuous">
@@ -364,5 +367,5 @@
             <child link="middle_wheel_link_${prefix}"/>
             <axis xyz="0 1 0"/>
-            <velocity>5.0</velocity>
+            <limit effort="100.0" velocity="5.0"/>
         </joint>
         <link name="rear_wheel_link_${prefix}">
@@ -387,6 +390,6 @@
         </link>
         <gazebo reference="rear_wheel_link_${prefix}">
-            <mu1>2.0</mu1>
-            <mu2>2.0</mu2>
+            <mu1>0.7</mu1>
+            <mu2>0.05</mu2>
         </gazebo>
         <joint name="rear_wheel_joint_${prefix}" type="continuous">
@@ -395,5 +398,5 @@
             <child link="rear_wheel_link_${prefix}"/>
             <axis xyz="0 1 0"/>
-            <velocity>5.0</velocity>
+            <limit effort="100.0" velocity="5.0"/>
         </joint>
     </xacro:macro>
@@ -405,5 +408,11 @@
         <origin xyz="0 0 0" rpy="0 0 0"/>
     </joint>
-    <link name="imu_link"></link>
+    <link name="imu_link">
+        <inertial>
+            <mass value="0.01"/>
+            <origin xyz="0 0 0" rpy="0 0 0"/>
+            <inertia ixx="0.0001" ixy="0" ixz="0" iyy="0.0001" iyz="0" izz="0.0001"/>
+        </inertial>
+    </link>
     <link name="laser_frame">
         <visual>
